File: MCU.kicad_sch (KiCad schematic)
At the start: 12 parts, among them P2 CONN_01X02, U1 STM32G0B1CBT, X3 TC2030-NL, Y1 830108313809

Commit message: clean up
Parts:
- C1, C2, C3, C4, C5: footprint Capacitors_SMD:C_0603 -> Capacitor_SMD:C_0603_1608Metric
- P2: footprint Connector_generic:Header_1x2_Pitch2.54mm -> Jumper:SolderJumper-2_P1.3mm_Open_RoundedPad1.0x1.5mm; now fitted
- R6: footprint Resistors_SMD:R_0603 -> Resistor_SMD:R_0603_1608Metric
- TP4, TP5: footprint Connector_generic:TP1.0mm -> TestPoint:TestPoint_Pad_1.0x1.0mm
- U1: footprint QFP:LQFP-48_7mmx7mm_Pitch0.5mm -> Package_QFP:LQFP-48_7x7mm_P0.5mm; Datasheet2 $PTX_DATASHEETS/datasheets/Microcontroller/STW_stm32g0b1re_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 -> https://www.st.com/resource/en/user_manual/um3083-stm32g0-s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; mouser (none) -> 511-STM32G0B1CBT3
- Y1: footprint crystal:Crystal_4Pin_SMD_3.2mmx2.5mm -> Crystal:Crystal_SMD_3225-4Pin_3.2x2.5mm
Connections:
- net CAN1_S: no longer names the net of U1.37 (PA15)
- net CAN2_S: no longer names the net of U1.21 (PB2)
- no-connect marks 28 -> 30

Commit message: gsi-v1
Parts:
- removed C4: 100n, Capacitor_SMD:C_0603_1608Metric, symbol multicomp:100n
- removed TP4, TP5: TP1.0mm, TestPoint:TestPoint_Pad_1.0x1.0mm, symbol generic-connectors:TP1.0mm
- C3, C5: MPN MC0603B104K500CT -> any; note (none) -> stock
- R6: MPN any -> (none)
- U1: digikey (none) -> 497-STM32G0B1CBT6-ND
- Y1: digikey (none) -> 732-830108313809CT-ND; mouser (none) -> 710-830108313809
Connections:
- net RX: no longer names the net of U1.32 (PA10)
- net TX: no longer names the net of U1.29 (PA9)
- no-connect marks 30 -> 32
Other:
- moved on the sheet: C5

Commit message: ready for production
Parts:
- C1, C2: value 6p2_0603_C0G_5%_50V_-40C..125C_Chip-Capacitor -> 6p2; MPN any -> CC0603BRNPO9BN6R2; digikey (none) -> 13-CC0603BRNPO9BN6R2CT-ND; note (none) -> candlelight
- C3, C5: note stock -> candlelight; now left out of the parts list
- P2, X3: note (none) -> candlelight; now left out of the parts list
- R6: value 10k_0603_100mW_1%_E24_Chip-Resistor -> 10k; note (none) -> candlelight; now left out of the parts list
- U1, Y1: note (none) -> candlelight
Changed lines of the file:
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@@
 			)
 		)
-		(property "note" ""
+		(property "note" "candlelight"
 			(at 173.99 25.4 0)
 			(effects
@@
 			)
 		)
-		(property "Value" "6p2_0603_C0G_5%_50V_-40C..125C_Chip-Capacitor"
+		(property "Value" "6p2"
 			(at 141.605 114.3 0)
 			(effects
@@
 			)
 		)
-		(property "MPN" "any"
+		(property "MPN" "CC0603BRNPO9BN6R2"
 			(at 139.065 121.92 0)
 			(effects
@@
 			)
 		)
-		(property "note" ""
+		(property "note" "candlelight"
+			(at 142.24 116.84 0)
+			(effects
+				(font
+					(size 1.27 1.27)
+				)
+				(hide yes)
+			)
+		)
+		(property "digikey" "13-CC0603BRNPO9BN6R2CT-ND"
 			(at 142.24 116.84 0)
 			(effects
@@
 		(unit 1)
 		(exclude_from_sim no)
-		(in_bom yes)
+		(in_bom no)
 		(on_board yes)
 		(dnp no)
@@
 			)
 		)
-		(property "note" ""
+		(property "note" "candlelight"
 			(at 36.83 36.83 0)
 			(effects
@@
 			)
 		)
-		(property "note" ""
+		(property "note" "candlelight"
 			(at 177.8 49.53 0)
 			(effects
@@
 		(unit 1)
 		(exclude_from_sim no)
-		(in_bom yes)
+		(in_bom no)
 		(on_board yes)
 		(dnp no)
@@
 			)
 		)
-		(property "note" ""
+		(property "note" "candlelight"
 			(at 35.56 60.96 0)
 			(effects
@@
 			)
 		)
-		(property "note" ""
+		(property "note" "candlelight"
 			(at 176.53 105.41 0)
 			(effects
@@
 		(unit 1)
 		(exclude_from_sim no)
-		(in_bom yes)
+		(in_bom no)
 		(on_board yes)
 		(dnp no)
@@
 			)
 		)
-		(property "Datasheet" "http://www.farnell.com/datasheets/1901289.pdf"
+		(property "Datasheet" ""
 			(at 149.606 88.519 0)
 			(effects
@@
 			)
 		)
-		(property "note" "stock"
+		(property "note" "candlelight"
 			(at 146.05 82.55 0)
 			(effects
@@
 		(unit 1)
 		(exclude_from_sim no)
-		(in_bom yes)
+		(in_bom no)
 		(on_board yes)
 		(dnp no)
@@
 			)
 		)
-		(property "Value" "10k_0603_100mW_1%_E24_Chip-Resistor"
+		(property "Value" "10k"
 			(at 37.1856 69.8246 90)
 			(effects
@@
 			)
 		)
-		(property "note" ""
+		(property "note" "candlelight"
 			(at 40.64 69.85 0)
 			(effects
@@
 			)
 		)
-		(property "note" ""
+		(property "note" "candlelight"
 			(at 176.53 82.55 0)
 			(effects
@@
 			)
 		)
-		(property "note" ""
+		(property "note" "candlelight"
 			(at 134.62 111.76 0)
 			(effects
@@
 			)
 		)
-		(property "note" ""
+		(property "note" "candlelight"
 			(at 128.27 39.37 0)
 			(effects
@@
 		(unit 1)
 		(exclude_from_sim no)
-		(in_bom yes)
+		(in_bom no)
 		(on_board yes)
 		(dnp no)
@@
 			)
 		)
-		(property "Datasheet" "http://www.farnell.com/datasheets/1901289.pdf"
+		(property "Datasheet" ""
 			(at 157.226 118.999 0)
 			(effects
@@
 			)
 		)
-		(property "note" "stock"
+		(property "note" "candlelight"
 			(at 153.67 113.03 0)
 			(effects
@@
 			)
 		)
-		(property "Value" "6p2_0603_C0G_5%_50V_-40C..125C_Chip-Capacitor"
+		(property "Value" "6p2"
 			(at 126.365 114.3 0)
 			(effects
@@
 			)
 		)
-		(property "MPN" "any"
+		(property "MPN" "CC0603BRNPO9BN6R2"
 			(at 123.825 121.92 0)
 			(effects
@@
 			)
 		)
-		(property "note" ""
+		(property "note" "candlelight"
+			(at 127 116.84 0)
+			(effects
+				(font
+					(size 1.27 1.27)
+				)
+				(hide yes)
+			)
+		)
+		(property "digikey" "13-CC0603BRNPO9BN6R2CT-ND"
 			(at 127 116.84 0)
 			(effects
@@
 			)
 		)
-		(property "note" ""
+		(property "note" "candlelight"
 			(at 81.28 40.64 0)
 			(effects
