File: candleLightfd-S01.kicad_sch (KiCad schematic)
At the start: 19 parts, among them P1 CONN_01X02, T101 Tab, T102 Tab, T103 Tab, T104 Tab, X1 629722000214_pasteInHole

Commit message: clean up
Parts:
- removed NB2: LAYERSTACK_TB, mechanical:LAYERSTACK_TB, symbol mechanical:LAYERSTACK_TB
- removed NB3, NB4: Passermarke_1mm_1.8mmx1.8mm, mechanical:Passermarke_1mm_1.8mmx1.8mm, symbol mechanical:Passermarke_1mm_1.8mmx1.8mm
- removed P1: CONN_01X02, Connector_generic:Header_1x2_Pitch2.54mm, symbol generic-connectors:CONN_01X02
- removed R1, R2: 5k1_0603_100mW_1%_E24_Chip-Resistor, Resistors_SMD:R_0603, symbol Res_1Percent_E24_0603_100mW_-40C-90C:5k1_0603_100mW_1%_E24_Chip-Resistor
- removed T101, T102, T103, T104: Tab, kikit:Tab, symbol kikit:Tab
- removed X1: 629722000214_pasteInHole, Socket_GCT:USB4105_pasteInHole, symbol wuerth:629722000214_pasteInHole
- removed X2: ~, d-sub:D-SUB-9_side, symbol d-sub:D-SUB-9_side
- added J1: CAN1, Connector_PinHeader_2.54mm:PinHeader_1x04_P2.54mm_Horizontal, symbol Connector_Generic:Conn_01x04
- added J2: CAN2, Connector_PinHeader_2.54mm:PinHeader_1x04_P2.54mm_Horizontal, symbol Connector_Generic:Conn_01x04
- added J3: USB_C_Receptacle_USB2.0_16P, Connector_USB:USB_C_Receptacle_GCT_USB4085, symbol Connector:USB_C_Receptacle_USB2.0_16P
- added R10, R9: 5k1_0603_100mW_1%_E24_Chip-Resistor, Resistor_SMD:R_0603_1608Metric, symbol Res_1Percent_E24_0603_100mW_-40C-90C:5k1_0603_100mW_1%_E24_Chip-Resistor
- D1, D2, D3: footprint LEDs_Kingbright:LED_Kingbright_0603 -> LED_SMD:LED_0603_1608Metric
- R3, R4, R5: footprint Resistors_SMD:R_0603 -> Resistor_SMD:R_0603_1608Metric
Connections:
- net +5V: now also J3.A4 (VBUS), J3.A9 (VBUS), J3.B4 (VBUS), J3.B9 (VBUS)
- net CAN1_H: now also J1.3 (Pin_3)
- net CAN1_L: now also J1.4 (Pin_4)
- net CAN2_H: now also J2.3 (Pin_3)
- net CAN2_L: now also J2.4 (Pin_4)
- net GND: now also J3.A1 (GND), J3.A12 (GND), J3.B1 (GND), J3.B12 (GND), J3.S1 (SHIELD), R10.2, R9.2
- net USB_N: now also J3.A7 (D-), J3.B7 (D-)
- net USB_P: now also J3.A6 (D+), J3.B6 (D+)
- new net: J3.B5 (CC2), R9.1
- new net: J3.A5 (CC1), R10.1
- new net GNDD: J1.2 (Pin_2), J2.2 (Pin_2)
Other:
- sheet CAN Transceiver ports: added none; removed CAN1_S, CAN2_S
- sheet MCU ports: added none; removed CAN1_S, CAN2_S
- moved on the sheet: NB1

Commit message: gsi-v1
Parts:
- J3: MPN (none) -> GSB1C411111DS1HR; digikey (none) -> 664-GSB1C411111DS1HRCT-ND; mfr GSB1C411111DS1HR -> (none)
- R10, R3, R4, R5, R9: MPN any -> (none)
Changed lines of the file:
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@@
+			)
+		)
+		(property "note" ""
+			(at 242.57 74.93 0)
+			(effects
+				(font
+					(size 1.27 1.27)
+				)
+				(hide yes)
 			)
 		)
@@
 			)
 		)
-		(property "MPN" "any"
+		(property "MPN" ""
 			(at 216.662 116.84 90)
 			(effects
@@
 				(font
 					(size 0.635 0.635)
+				)
+				(hide yes)
+			)
+		)
+		(property "note" ""
+			(at 212.09 119.38 0)
+			(effects
+				(font
+					(size 1.27 1.27)
 				)
 				(hide yes)
@@
 			)
 		)
-		(property "MPN" "any"
+		(property "MPN" ""
 			(at 61.722 73.66 90)
 			(effects
@@
 				(font
 					(size 0.635 0.635)
+				)
+				(hide yes)
+			)
+		)
+		(property "note" ""
+			(at 57.15 76.2 0)
+			(effects
+				(font
+					(size 1.27 1.27)
 				)
 				(hide yes)
@@
 			)
 		)
-		(property "Datasheet" "$PTX_DATASHEETS/datasheets/LED/Kingbright_KPT-1608SGC.pdf"
+		(property "Datasheet" ""
 			(at 218.44 124.46 0)
 			(effects
@@
 		)
 		(property "Field10" ""
+			(at 212.09 128.27 0)
+			(effects
+				(font
+					(size 1.27 1.27)
+				)
+				(hide yes)
+			)
+		)
+		(property "note" ""
 			(at 212.09 128.27 0)
 			(effects
@@
 			)
 		)
+		(property "note" ""
+			(at 124.46 27.94 0)
+			(effects
+				(font
+					(size 1.27 1.27)
+				)
+				(hide yes)
+			)
+		)
 		(instances
 			(project "candleLightfd-S01"
@@
 			)
 		)
-		(property "MPN" "any"
+		(property "MPN" ""
 			(at 69.342 73.66 90)
 			(effects
@@
 				(font
 					(size 0.635 0.635)
+				)
+				(hide yes)
+			)
+		)
+		(property "note" ""
+			(at 64.77 76.2 0)
+			(effects
+				(font
+					(size 1.27 1.27)
 				)
 				(hide yes)
@@
 			)
 		)
-		(property "mfr" "GSB1C411111DS1HR "
+		(property "mouser" " 523-GSB1C411111DS1HR "
 			(at 30.48 77.47 0)
 			(effects
@@
 			)
 		)
-		(property "mouser" " 523-GSB1C411111DS1HR "
+		(property "digikey" "664-GSB1C411111DS1HRCT-ND"
+			(at 30.48 77.47 0)
+			(effects
+				(font
+					(size 1.27 1.27)
+				)
+				(hide yes)
+			)
+		)
+		(property "MPN" "GSB1C411111DS1HR "
+			(at 30.48 77.47 0)
+			(effects
+				(font
+					(size 1.27 1.27)
+				)
+				(hide yes)
+			)
+		)
+		(property "note" ""
 			(at 30.48 77.47 0)
 			(effects
@@
 			)
 		)
-		(property "MPN" "any"
+		(property "MPN" ""
 			(at 236.982 116.84 90)
 			(effects
@@
 				(font
 					(size 0.635 0.635)
+				)
+				(hide yes)
+			)
+		)
+		(property "note" ""
+			(at 232.41 119.38 0)
+			(effects
+				(font
+					(size 1.27 1.27)
 				)
 				(hide yes)
@@
 			)
 		)
-		(property "Datasheet" "$PTX_DATASHEETS/datasheets/LED/Kingbright_KPT-1608EC.pdf"
+		(property "Datasheet" ""
 			(at 259.08 124.46 0)
 			(effects
@@
 		)
 		(property "Field10" ""
+			(at 252.73 128.27 0)
+			(effects
+				(font
+					(size 1.27 1.27)
+				)
+				(hide yes)
+			)
+		)
+		(property "note" ""
 			(at 252.73 128.27 0)
 			(effects
@@
 			)
 		)
-		(property "Datasheet" "$PTX_DATASHEETS/datasheets/LED/Kingbright_KPT-1608SGC.pdf"
+		(property "Datasheet" ""
 			(at 238.76 124.46 0)
 			(effects
@@
 		)
 		(property "Field10" ""
+			(at 232.41 128.27 0)
+			(effects
+				(font
+					(size 1.27 1.27)
+				)
+				(hide yes)
+			)
+		)
+		(property "note" ""
 			(at 232.41 128.27 0)
 			(effects
@@
 			)
 		)
-		(property "MPN" "any"
+		(property "MPN" ""
 			(at 257.302 116.84 90)
 			(effects
@@
 				(font
 					(size 0.635 0.635)
+				)
+				(hide yes)
+			)
+		)
+		(property "note" ""
+			(at 252.73 119.38 0)
+			(effects
+				(font
+					(size 1.27 1.27)
 				)
 				(hide yes)
@@
 			(at 242.57 54.61 0)
 			(effects
+				(font
+					(size 1.27 1.27)
+				)
+				(hide yes)
+			)
+		)
+		(property "note" ""
+			(at 242.57 54.61 0)
+			(effects

Commit message: replace connector CAN1/2 with PSS
Parts:
- J1, J2: footprint Connector_PinHeader_2.54mm:PinHeader_1x04_P2.54mm_Horizontal -> Connector_PSS254:PSS254_1x04_Horizontal
Changed lines of the file:
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@@
 			)
 		)
-		(property "Footprint" "Connector_PinHeader_2.54mm:PinHeader_1x04_P2.54mm_Horizontal"
+		(property "Footprint" "Connector_PSS254:PSS254_1x04_Horizontal"
 			(at 242.57 74.93 0)
 			(effects
@@
 			)
 		)
-		(property "Footprint" "Connector_PinHeader_2.54mm:PinHeader_1x04_P2.54mm_Horizontal"
+		(property "Footprint" "Connector_PSS254:PSS254_1x04_Horizontal"
 			(at 242.57 54.61 0)
 			(effects

Commit message: ready for production
Parts:
- D1, D2, D3, J1, J2, NB1: note (none) -> candlelight; now left out of the parts list
- J3: note (none) -> candlelight
- R10, R9: value 5k1_0603_100mW_1%_E24_Chip-Resistor -> 5k1; note (none) -> candlelight; now left out of the parts list
- R3, R4, R5: value 1k_0603_100mW_1%_E24_Chip-Resistor -> 1k; note (none) -> candlelight; now left out of the parts list
Changed lines of the file:
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@@
 		(unit 1)
 		(exclude_from_sim no)
-		(in_bom yes)
+		(in_bom no)
 		(on_board yes)
 		(dnp no)
@@
 			)
 		)
-		(property "note" ""
+		(property "note" "candlelight"
 			(at 242.57 74.93 0)
 			(effects
@@
 		(unit 1)
 		(exclude_from_sim no)
-		(in_bom yes)
+		(in_bom no)
 		(on_board yes)
 		(dnp no)
@@
 			)
 		)
-		(property "Value" "1k_0603_100mW_1%_E24_Chip-Resistor"
+		(property "Value" "1k"
 			(at 208.6356 119.3546 90)
 			(effects
@@
 			)
 		)
-		(property "note" ""
+		(property "note" "candlelight"
 			(at 212.09 119.38 0)
 			(effects
@@
 		(unit 1)
 		(exclude_from_sim no)
-		(in_bom yes)
+		(in_bom no)
 		(on_board yes)
 		(dnp no)
@@
 			)
 		)
-		(property "Value" "5k1_0603_100mW_1%_E24_Chip-Resistor"
+		(property "Value" "5k1"
 			(at 53.6956 76.1746 90)
 			(effects
@@
 			)
 		)
-		(property "note" ""
+		(property "note" "candlelight"
 			(at 57.15 76.2 0)
 			(effects
@@
 		(unit 1)
 		(exclude_from_sim no)
-		(in_bom yes)
+		(in_bom no)
 		(on_board yes)
 		(dnp no)
@@
 			)
 		)
-		(property "note" ""
+		(property "note" "candlelight"
 			(at 212.09 128.27 0)
 			(effects
@@
 		(unit 1)
 		(exclude_from_sim no)
-		(in_bom yes)
+		(in_bom no)
 		(on_board yes)
 		(dnp no)
@@
 			)
 		)
-		(property "note" ""
+		(property "note" "candlelight"
 			(at 124.46 27.94 0)
 			(effects
@@
 		(unit 1)
 		(exclude_from_sim no)
-		(in_bom yes)
+		(in_bom no)
 		(on_board yes)
 		(dnp no)
@@
 			)
 		)
-		(property "Value" "5k1_0603_100mW_1%_E24_Chip-Resistor"
+		(property "Value" "5k1"
 			(at 61.3156 76.1746 90)
 			(effects
@@
 			)
 		)
-		(property "note" ""
+		(property "note" "candlelight"
 			(at 64.77 76.2 0)
 			(effects
@@
 			)
 		)
-		(property "note" ""
+		(property "note" "candlelight"
 			(at 30.48 77.47 0)
 			(effects
@@
 		(unit 1)
 		(exclude_from_sim no)
-		(in_bom yes)
+		(in_bom no)
 		(on_board yes)
 		(dnp no)
@@
 			)
 		)
-		(property "Value" "1k_0603_100mW_1%_E24_Chip-Resistor"
+		(property "Value" "1k"
 			(at 228.9556 119.3546 90)
 			(effects
@@
 			)
 		)
-		(property "note" ""
+		(property "note" "candlelight"
 			(at 232.41 119.38 0)
 			(effects
@@
 		(unit 1)
 		(exclude_from_sim no)
-		(in_bom yes)
+		(in_bom no)
 		(on_board yes)
 		(dnp no)
@@
 			)
 		)
-		(property "note" ""
+		(property "note" "candlelight"
 			(at 252.73 128.27 0)
 			(effects
@@
 		(unit 1)
 		(exclude_from_sim no)
-		(in_bom yes)
+		(in_bom no)
 		(on_board yes)
 		(dnp no)
@@
 			)
 		)
-		(property "note" ""
+		(property "note" "candlelight"
 			(at 232.41 128.27 0)
 			(effects
@@
 		(unit 1)
 		(exclude_from_sim no)
-		(in_bom yes)
+		(in_bom no)
 		(on_board yes)
 		(dnp no)
@@
 			)
 		)
-		(property "Value" "1k_0603_100mW_1%_E24_Chip-Resistor"
+		(property "Value" "1k"
 			(at 249.2756 119.3546 90)
 			(effects
@@
 			)
 		)
-		(property "note" ""
+		(property "note" "candlelight"
 			(at 252.73 119.38 0)
 			(effects
@@
 		(unit 1)
 		(exclude_from_sim no)
-		(in_bom yes)
+		(in_bom no)
 		(on_board yes)
 		(dnp no)
@@
 			)
 		)
-		(property "note" ""
+		(property "note" "candlelight"
 			(at 242.57 54.61 0)
 			(effects
