File: transceiver.kicad_sch (KiCad schematic)
At the start: 8 parts, among them U1 TJA1051T3

Commit message: clean up
Parts:
- removed C7 (x2), C8 (x2): 100n_0603_X7R_10%_50V_-40C..125C_Chip-Capacitor, Capacitors_SMD:C_0603, symbol Cap_10Percent_E24_0603_X7R_50V_-40C-125C:100n_0603_X7R_10%_50V_-40C..125C_Chip-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
- removed R5 (x2): 120R_0805_125mW_1%_E24_Chip-Resistor, Resistors_SMD:R_0805, symbol Res_1Percent_E24_0805_125mW_-40C-90C:120R_0805_125mW_1%_E24_Chip-Resistor
- removed U1 (x2): TJA1051T3, tssop:SOIC-8_3.90mmx4.90mm_Pitch1.27mm, symbol nxp:TJA1051T3
- added C12, C13: 100n_0603_X7R_10%_50V_-40C..125C_Chip-Capacitor, Capacitor_SMD:C_0603_1608Metric, symbol Cap_10Percent_E24_0603_X7R_50V_-40C-125C:100n_0603_X7R_10%_50V_-40C..125C_Chip-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
- added R7, R8: 120, Resistor_SMD:R_0603_1608Metric, symbol Device:R
- added SW1: Term1, Button_Switch_THT:SW_Slide_SPDT_Angled_CK_OS102011MA1Q, symbol Switch:SW_SPDT
- added SW2: Term2, Button_Switch_THT:SW_Slide_SPDT_Angled_CK_OS102011MA1Q, symbol Switch:SW_SPDT
- added U5, U6: ISO1044BD, Package_SO:SOIC-8_3.9x4.9mm_P1.27mm, symbol Interface_CAN_LIN:ISO1044BD
- added U7: NXE1S0505MC, Converter_DCDC:Converter_DCDC_Murata_NXExSxxxxMC_SMD, symbol Regulator_Switching:NXE1S0505MC
Connections:
- net +3V3: now also C12.1, C13.1, U5.1 (VCC1), U6.1 (VCC1)
- net +5V: now also U7.3 (+VIN)
- net CAN1_H: now also R7.1, U5.6 (CANH)
- net CAN1_L: now also SW1.1 (A), U5.5 (CANL)
- net CAN1_RX: now also U5.3 (RXD)
- net CAN1_TX: now also U5.2 (TXD)
- net CAN2_H: now also R8.1, U6.6 (CANH)
- net CAN2_L: now also SW2.1 (A), U6.5 (CANL)
- net CAN2_RX: now also U6.3 (RXD)
- net CAN2_TX: now also U6.2 (TXD)
- net GND: now also C12.2, C13.2, U5.4 (GND1), U6.4 (GND1), U7.1 (-VIN)
- new net: R7.2, SW1.2 (B)
- new net: R8.2, SW2.2 (B)
- new net +5VD: U5.8 (VCC2), U6.8 (VCC2), U7.8 (+VOUT)
- new net GNDD: U5.7 (GND2), U6.7 (GND2), U7.7 (-VOUT)

Commit message: gsi-v1
Parts:
- removed U6: ISO1044BD, Package_SO:SOIC-8_3.9x4.9mm_P1.27mm, symbol Interface_CAN_LIN:ISO1044BD
- removed U7: NXE1S0505MC, Converter_DCDC:Converter_DCDC_Murata_NXExSxxxxMC_SMD, symbol Regulator_Switching:NXE1S0505MC
- added C10, C8: 10u_0603_X7R_10%_50V_-40C..125C_Chip-Capacitor, Capacitor_SMD:C_0603_1608Metric, symbol Cap_10Percent_E24_0603_X7R_50V_-40C-125C:100n_0603_X7R_10%_50V_-40C..125C_Chip-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
- added C11, C9: 100n_0603_X7R_10%_50V_-40C..125C_Chip-Capacitor, Capacitor_SMD:C_0603_1608Metric, symbol Cap_10Percent_E24_0603_X7R_50V_-40C-125C:100n_0603_X7R_10%_50V_-40C..125C_Chip-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
- added U3: R05CTE05S, Package_SO:SOIC-16W_7.5x10.3mm_P1.27mm, symbol DCDC_Recom:R05CTE05S
- added U4: ISO1044BD, Package_SO:SOIC-8_3.9x4.9mm_P1.27mm, symbol Interface_CAN_LIN:ISO1044BD
- SW1, SW2: MPN (none) -> OS102011MA1QS1; digikey (none) -> CKN9560-ND
- U5: MPN (none) -> ISO1044BDR; digikey (none) -> 296-ISO1044BDRCT-ND
Connections:
- net +3V3: now also U4.1 (VCC1)
- net +5V: now also C10.1, C11.1, U3.3 (+VIN), U3.4 (+VIN)
- net +5VD: now also C8.1, C9.1, U3.13 (+VOUT), U3.14 (+VOUT), U4.8 (VCC2)
- net CAN1_H: now also U4.6 (CANH); no longer U5.6 (CANH)
- net CAN1_L: now also SW1.2 (B), U4.5 (CANL); no longer SW1.1 (A), U5.5 (CANL)
- net CAN1_RX: now also U4.3 (RXD); no longer U5.3 (RXD)
- net CAN1_TX: now also U4.2 (TXD); no longer U5.2 (TXD)
- net CAN2_H: now also U5.6 (CANH)
- net CAN2_L: now also SW2.2 (B), U5.5 (CANL); no longer SW2.1 (A)
- net CAN2_RX: now also U5.3 (RXD)
- net CAN2_TX: now also U5.2 (TXD)
- net GNDD: now also C8.2, C9.2, U3.11 (SGNDout), U3.12 (SGNDout), U3.15 (-VOUT), U3.16 (-VOUT), U3.9 (SGNDout), U4.7 (GND2)
- net at R7.2: now also SW1.3 (C); no longer SW1.2 (B)
- net at R8.2: now also SW2.1 (A); no longer SW2.2 (B)
- net GND renamed -VIN
- net -VIN: now also C10.2, C11.2, U3.1 (-VIN), U3.2 (-VIN), U3.5 (SGNDin), U3.6 (SGNDin), U3.7 (SGNDin), U3.8 (SGNDin), U4.4 (GND1)
Other:
- moved on the sheet: SW1, U5

Commit message: ready for production
Parts:
- C10, C8: value 10u_0603_X7R_10%_50V_-40C..125C_Chip-Capacitor -> 10u; note (none) -> candlelight; now left out of the parts list
- C11, C12, C13, C9: value 100n_0603_X7R_10%_50V_-40C..125C_Chip-Capacitor -> 100n; note (none) -> candlelight; now left out of the parts list
- R7, R8: note (none) -> candlelight; now left out of the parts list
- SW1, SW2, U3, U4, U5: note (none) -> candlelight
Changed lines of the file:
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@@
 		(unit 1)
 		(exclude_from_sim no)
-		(in_bom yes)
+		(in_bom no)
 		(on_board yes)
 		(dnp no)
@@
 			)
 		)
-		(property "Value" "100n_0603_X7R_10%_50V_-40C..125C_Chip-Capacitor"
+		(property "Value" "100n"
 			(at 144.145 64.77 0)
 			(effects
@@
 			)
 		)
-		(property "note" ""
+		(property "note" "candlelight"
 			(at 143.51 62.23 0)
 			(effects
@@
 			)
 		)
-		(property "note" ""
+		(property "note" "candlelight"
 			(at 162.56 104.14 0)
 			(effects
@@
 			)
 		)
-		(property "note" ""
+		(property "note" "candlelight"
 			(at 110.49 62.23 0)
 			(effects
@@
 		(unit 1)
 		(exclude_from_sim no)
-		(in_bom yes)
+		(in_bom no)
 		(on_board yes)
 		(dnp no)
@@
 			)
 		)
-		(property "Value" "100n_0603_X7R_10%_50V_-40C..125C_Chip-Capacitor"
+		(property "Value" "100n"
 			(at 76.835 99.06 0)
 			(effects
@@
 			)
 		)
-		(property "note" ""
+		(property "note" "candlelight"
 			(at 76.2 96.52 0)
 			(effects
@@
 		(unit 1)
 		(exclude_from_sim no)
-		(in_bom yes)
+		(in_bom no)
 		(on_board yes)
 		(dnp no)
@@
 			)
 		)
-		(property "note" ""
+		(property "note" "candlelight"
 			(at 165.1 92.71 0)
 			(effects
@@
 		(unit 1)
 		(exclude_from_sim no)
-		(in_bom yes)
+		(in_bom no)
 		(on_board yes)
 		(dnp no)
@@
 			)
 		)
-		(property "Value" "100n_0603_X7R_10%_50V_-40C..125C_Chip-Capacitor"
+		(property "Value" "100n"
 			(at 76.835 64.77 0)
 			(effects
@@
 			)
 		)
-		(property "note" ""
+		(property "note" "candlelight"
 			(at 77.47 62.23 0)
 			(effects
@@
 		(unit 1)
 		(exclude_from_sim no)
-		(in_bom yes)
+		(in_bom no)
 		(on_board yes)
 		(dnp no)
@@
 			)
 		)
-		(property "Value" "10u_0603_X7R_10%_50V_-40C..125C_Chip-Capacitor"
+		(property "Value" "10u"
 			(at 88.265 64.77 0)
 			(effects
@@
 			)
 		)
-		(property "note" ""
+		(property "note" "candlelight"
 			(at 88.9 62.23 0)
 			(effects
@@
 			)
 		)
-		(property "note" ""
+		(property "note" "candlelight"
 			(at 110.49 130.81 0)
 			(effects
@@
 			)
 		)
-		(property "note" ""
+		(property "note" "candlelight"
 			(at 110.49 95.25 0)
 			(effects
@@
 			)
 		)
-		(property "note" ""
+		(property "note" "candlelight"
 			(at 167.64 138.43 0)
 			(effects
@@
 		(unit 1)
 		(exclude_from_sim no)
-		(in_bom yes)
+		(in_bom no)
 		(on_board yes)
 		(dnp no)
@@
 			)
 		)
-		(property "Value" "100n_0603_X7R_10%_50V_-40C..125C_Chip-Capacitor"
+		(property "Value" "100n"
 			(at 76.835 134.62 0)
 			(effects
@@
 			)
 		)
-		(property "note" ""
+		(property "note" "candlelight"
 			(at 76.2 132.08 0)
 			(effects
@@
 		(unit 1)
 		(exclude_from_sim no)
-		(in_bom yes)
+		(in_bom no)
 		(on_board yes)
 		(dnp no)
@@
 			)
 		)
-		(property "note" ""
+		(property "note" "candlelight"
 			(at 165.1 127 0)
 			(effects
@@
 		(unit 1)
 		(exclude_from_sim no)
-		(in_bom yes)
+		(in_bom no)
 		(on_board yes)
 		(dnp no)
@@
 			)
 		)
-		(property "Value" "10u_0603_X7R_10%_50V_-40C..125C_Chip-Capacitor"
+		(property "Value" "10u"
 			(at 132.715 64.77 0)
 			(effects
@@
 			)
 		)
-		(property "note" ""
+		(property "note" "candlelight"
 			(at 132.08 62.23 0)
 			(effects
